File: schematics/whenisbins/whenisbins.kicad_pcb (KiCad board)
At the start: 2 copper layers, 73 x 54.5 mm, 28 parts, among them J1 Raspberry Pi Header, J10 Bin 2, J11 Bin 3, J12 Bin 4, J13 LCD Pins, J2 PIR, J3 Bin 1 LED, J4 Bin 2 LED, J5 Bin 3 LED, J6 Bin 4 LED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

Commit message: Finalise pcb and set up selenium
Parts:
- added H1: MH, MountingHole:MountingHole_2.5mm_Pad_TopBottom, F.Cu at (176.2, 122.2)
- added H2: MH, MountingHole:MountingHole_2.5mm_Pad_TopBottom, F.Cu at (109.8, 122.2)
- added H3: MH, MountingHole:MountingHole_2.5mm_Pad_TopBottom, F.Cu at (176.2, 89.5)
- added H4: MH, MountingHole:MountingHole_2.5mm_Pad_TopBottom, F.Cu at (109.8, 89.5)
- added J14: Bin 5, Connector_PinHeader_2.54mm:PinHeader_1x02_P2.54mm_Vertical, F.Cu at (172.5, 95.0)
- added J15: Bin 6, Connector_PinHeader_2.54mm:PinHeader_1x02_P2.54mm_Vertical, F.Cu at (168.5, 95.0)
- added J16: Bin 7, Connector_PinHeader_2.54mm:PinHeader_1x02_P2.54mm_Vertical, F.Cu at (164.5, 95.0)
- added J17: Bin 5 LED, Connector_PinHeader_2.54mm:PinHeader_1x02_P2.54mm_Vertical, F.Cu at (160.5, 95.0)
- added J18: Bin 6 LED, Connector_PinHeader_2.54mm:PinHeader_1x02_P2.54mm_Vertical, F.Cu at (156.5, 95.0)
- added J19: Bin 7 LED, Connector_PinHeader_2.54mm:PinHeader_1x02_P2.54mm_Vertical, F.Cu at (152.5, 95.0)
- added R13: 220Ω, Resistor_THT:R_Axial_DIN0207_L6.3mm_D2.5mm_P10.16mm_Horizontal, F.Cu at (172.5, 111.6)
- added R14: 220Ω, Resistor_THT:R_Axial_DIN0207_L6.3mm_D2.5mm_P10.16mm_Horizontal, F.Cu at (168.5, 111.6)
- added R15: 220Ω, Resistor_THT:R_Axial_DIN0207_L6.3mm_D2.5mm_P10.16mm_Horizontal, F.Cu at (164.5, 111.5)
- added R16: 560Ω, Resistor_THT:R_Axial_DIN0207_L6.3mm_D2.5mm_P10.16mm_Horizontal, F.Cu at (160.5, 101.4)
- added R17: 560Ω, Resistor_THT:R_Axial_DIN0207_L6.3mm_D2.5mm_P10.16mm_Horizontal, F.Cu at (156.5, 101.4)
- added R18: 560Ω, Resistor_THT:R_Axial_DIN0207_L6.3mm_D2.5mm_P10.16mm_Horizontal, F.Cu at (152.5, 101.4)
- moved J2 43.1 mm to (154.5, 126.5), turned to 90 degrees
- moved R12 16.6 mm to (148.5, 111.5)
- moved J12 16.5 mm to (148.5, 95.0)
- moved R11 16.1 mm to (144.5, 111.5)
- moved J11 16.0 mm to (144.5, 95.0)
- moved R5 15.8 mm to (178.1, 127.5), turned to 180 degrees
- moved R10 15.6 mm to (140.5, 111.5)
- moved J10 15.5 mm to (140.5, 95.0)
- moved R9 15.1 mm to (136.5, 111.5)
- moved J9 15.0 mm to (136.5, 95.0)
- moved R8 14.6 mm to (132.5, 111.6)
- moved J7 14.5 mm to (132.5, 95.0)
- moved R7 14.1 mm to (128.5, 111.5)
- moved J8 14.0 mm to (128.5, 95.0)
- moved R4 12.7 mm to (124.5, 111.5)
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Connections:
- net /- renamed /GND
- J3 pad 2: /+ -> Net-(J3-Pin_2)
- J4 pad 2: /+ -> Net-(J4-Pin_2)
- J5 pad 2: /+ -> Net-(J5-Pin_2)
- J6 pad 2: /+ -> Net-(J6-Pin_2)
- R1 pad 2: /+ -> Net-(J3-Pin_2)
- R2 pad 2: /+ -> Net-(J4-Pin_2)
- R3 pad 2: /+ -> Net-(J5-Pin_2)
- R4 pad 2: /+ -> Net-(J6-Pin_2)
Routing:
- net /GND: track 0.00 -> 245.3 mm
- net /+3.3v: track 0.00 -> 117.6 mm
- net /+5V: track 0.00 -> 73.0 mm
- net /P11: track 0.00 -> 40.0 mm
- net /P10: track 0.00 -> 35.2 mm
- net /P05: track 0.00 -> 30.0 mm
- net /P26: track 0.00 -> 29.0 mm
- net /P06: track 0.00 -> 28.2 mm
- net /P13: track 0.00 -> 28.1 mm
- net /P19: track 0.00 -> 27.9 mm
- net /D4: track 0.00 -> 25.3 mm
- net /D5: track 0.00 -> 23.7 mm
- net /P16: track 0.00 -> 23.6 mm
- net /P18: track 0.00 -> 22.8 mm
- net /D6: track 0.00 -> 22.7 mm
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- added copper zone on B.Cu, net /GND
- added copper zone on F.Cu, net /GND
Other:
- board size 73 x 54.5 mm -> 73 x 55.5 mm
- board text added: "5 BTN"
- board text added: "6 BTN"
- board text added: "7 BTN"
- board text added: "B5 LED"
- board text added: "B6 LED"
- board text added: "B7 LED"
- board text added: "The Bin-Dicator v1"
