File: schematics/whenisbins/whenisbins.kicad_sch (KiCad schematic)
At the start: 28 parts, among them J1 Raspberry Pi Header, J10 Bin 2, J11 Bin 3, J12 Bin 4, J13 LCD Pins, J2 PIR, J3 Bin 1 LED, J4 Bin 2 LED, J5 Bin 3 LED, J6 Bin 4 LED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

Commit message: Finalise pcb and set up selenium
Parts:
- added H1, H2, H3, H4: MH, symbol Mechanical:MountingHole_Pad
- added J14: Bin 5, Connector_PinHeader_2.54mm:PinHeader_1x02_P2.54mm_Vertical, symbol Connector:Conn_01x02_Pin
- added J15: Bin 6, Connector_PinHeader_2.54mm:PinHeader_1x02_P2.54mm_Vertical, symbol Connector:Conn_01x02_Pin
- added J16: Bin 7, Connector_PinHeader_2.54mm:PinHeader_1x02_P2.54mm_Vertical, symbol Connector:Conn_01x02_Pin
- added J17: Bin 5 LED, Connector_PinHeader_2.54mm:PinHeader_1x02_P2.54mm_Vertical, symbol Connector:Conn_01x02_Pin
- added J18: Bin 6 LED, Connector_PinHeader_2.54mm:PinHeader_1x02_P2.54mm_Vertical, symbol Connector:Conn_01x02_Pin
- added J19: Bin 7 LED, Connector_PinHeader_2.54mm:PinHeader_1x02_P2.54mm_Vertical, symbol Connector:Conn_01x02_Pin
- added R13, R14, R15: 220Ω, Resistor_THT:R_Axial_DIN0207_L6.3mm_D2.5mm_P10.16mm_Horizontal, symbol Device:R
- added R16, R17, R18: 560Ω, Resistor_THT:R_Axial_DIN0207_L6.3mm_D2.5mm_P10.16mm_Horizontal, symbol Device:R
Connections:
- net +3.3v: now also J14.1 (Pin_1), J15.1 (Pin_1), J16.1 (Pin_1)
- net P05: now also R14.1
- net P06: now also R15.1
- net P11: now also R13.1
- net P13: now also R16.2
- net P19: now also R17.2
- net P26: now also R18.2
- removed net +: J3.2 (Pin_2), J4.2 (Pin_2), J5.2 (Pin_2), J6.2 (Pin_2), R1.2, R2.2, R3.2, R4.2
- net - renamed GND
- net GND: now also H1.1, H2.1, H3.1, H4.1, J17.1 (Pin_1), J18.1 (Pin_1), J19.1 (Pin_1)
- new net: J18.2 (Pin_2), R17.1
- new net: J5.2 (Pin_2), R3.2
- new net: J4.2 (Pin_2), R2.2
- new net: J6.2 (Pin_2), R4.2
- new net: J17.2 (Pin_2), R16.1
- new net: J16.2 (Pin_2), R15.2
- new net: J14.2 (Pin_2), R13.2
- new net: J3.2 (Pin_2), R1.2
- new net: J19.2 (Pin_2), R18.1
- new net: J15.2 (Pin_2), R14.2
- no-connect marks 16 -> 10
Other:
- note added: "+"
